Commit message: Robot spawns in Gazebo as well and the differential plugins are added as well

File: urdf/barista_robot_model.urdf (robot description, URDF)
Before this commit: robot rick, 10 links, 9 joints
Joints:
- joint base_link_to_back_caster: type continuous -> fixed
- joint base_link_to_front_caster: type continuous -> fixed
- joint base_link_to_left_wheel: limit (none) -> effort=10000 velocity=1000
- joint base_link_to_right_wheel: limit (none) -> effort=10000 velocity=1000

Commit message: Created the laser_scan using Hoyuko scanner. PART-1.

File: urdf/barista_robot_model.urdf (robot description, URDF)
Before this commit: robot rick, 10 links, 9 joints
Links:
- added link hokuyo_sensor, mass 0.160; collision box size=0.050 0.050 0.070; visual mesh filename=package://barista_robot_description/meshes/hokuyo_ust_10lx.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 scale=1 1 1
Joints:
- added joint base_link_to_hokuyo_sensor: type fixed, parent base_link, child hokuyo_sensor, origin xyz=0.130 0 0.0775 rpy=0 0 0
- joint base_link_to_left_wheel: origin xyz=0 -0.145 -0.0775 rpy=0 0 0 -> xyz=0 0.145 -0.0775 rpy=0 0 0
- joint base_link_to_right_wheel: origin xyz=0 0.145 -0.0775 rpy=0 0 0 -> xyz=0 -0.145 -0.0775 rpy=0 0 0
