Commit message: Created the caster.xacro and cup_holder_tray.xacro

File: xacro/barista_robot_model.urdf.xacro (robot description, xacro)
@@ -3,4 +3,6 @@
 <xacro:include filename="$(find barista_robot_description)/xacro/wheel.xacro" />
 <xacro:include filename="$(find barista_robot_description)/xacro/standoff.xacro" />
+<xacro:include filename="$(find barista_robot_description)/xacro/caster.xacro" />
+<xacro:include filename="$(find barista_robot_description)/xacro/cup_holder_tray.xacro" />
 <xacro:property name="base_link_radius" value="0.178"/>
 <xacro:property name="base_link_length" value="0.155"/>
@@ -39,18 +41,24 @@
 <!-- rod_d -->
 <xacro:standoff rod_name="rod_d" />
+<!-- front_caster -->
+<xacro:caster caster_name="front_caster" />
+<!-- back_caster -->
+<xacro:caster caster_name="back_caster" />
+<!-- cup_holder -->
+<xacro:cup_holder cup_holder_name="cup_holder" />
 <!-- joints -->
   <joint name="base_link_to_left_wheel" type="fixed">
-    <origin rpy="0 0 0" xyz="0 0.15 -0.0775"/>
+    <origin rpy="0 0 0" xyz="0 0.145 -0.0775"/>
     <child link="left_wheel"/>
     <parent link="base_link"/>
-    <axis rpy="0 0 0" xyz="0 1 0"/>
+    <axis rpy="0 0 0" xyz="0 0 1"/>
     <limit effort="1000" velocity="100"/>
     <joint_properties damping="1.0" friction="1.0"/>
   </joint>
   <joint name="base_link_to_right_wheel" type="fixed">
-    <origin rpy="0 0 0" xyz="0 -0.15 -0.0775"/>
+    <origin rpy="0 0 0" xyz="0 -0.145 -0.0775"/>
     <child link="right_wheel"/>
     <parent link="base_link"/>
-    <axis rpy="0 0 0" xyz="0 1 0"/>
+    <axis rpy="0 0 0" xyz="0 0 1"/>
     <limit effort="1000" velocity="100"/>
     <joint_properties damping="1.0" friction="1.0"/>
@@ -76,4 +84,23 @@
     <origin xyz="-0.040 -0.125 0.1875" rpy="0 0 0"/>
   </joint>
+  <joint name="base_link_to_front_caster" type="fixed">
+    <parent link="base_link"/>
+    <child link="front_caster"/>
+    <origin xyz="0.145 0 -0.09" rpy="0 0 0"/>
+    <axis xyz="0 1 0"/>
+    <joint_properties damping="1.0" friction="1.0"/>
+  </joint>
+  <joint name="base_link_to_back_caster" type="fixed">
+    <parent link="base_link"/>
+    <child link="back_caster"/>
+    <origin xyz="-0.145 0 -0.09" rpy="0 0 0"/>
+    <axis xyz="0 1 0"/>
+    <joint_properties damping="1.0" friction="1.0"/>
+  </joint>
+  <joint name="base_link_to_cup_holder" type="fixed">
+    <parent link="base_link"/>
+    <child link="cup_holder"/>
+    <origin xyz="0 0 0.330" rpy="0 0 0"/>
+  </joint>
 <!-- gazebo references -->
   <gazebo reference="right_wheel">
@@ -91,9 +118,23 @@
         <material>Gazebo/Black</material>
     </gazebo>
+<gazebo reference="front_caster">
+        <kp>1e6</kp>
+        <kd>10</kd>
+        <mu1>0.0</mu1>
+        <mu2>0.0</mu2>
+        <material>Gazebo/Black</material>
+    </gazebo>
+<gazebo reference="back_caster">
+        <kp>1e6</kp>
+        <kd>10</kd>
+        <mu1>0.0</mu1>
+        <mu2>0.0</mu2>
+        <material>Gazebo/Black</material>
+    </gazebo>
 <gazebo reference="base_link">
         <material>Gazebo/Red</material>
     </gazebo>
 <gazebo reference="cup_holder">
-        <material>Gazebo/Blue</material>
+        <material>Gazebo/Red</material>
     </gazebo>
 <gazebo reference="rod_a">
@@ -109,3 +150,9 @@
         <material>Gazebo/White</material>
     </gazebo>
+<gazebo reference="base_link_to_front_caster">
+        <preserveFixedJoint>true</preserveFixedJoint>
+    </gazebo>
+<gazebo reference="base_link_to_back_caster">
+        <preserveFixedJoint>true</preserveFixedJoint>
+    </gazebo>
 </robot>

File: xacro/wheel.xacro (robot description, xacro)
@@ -9,5 +9,5 @@
   <link name="${wheel_name}">
       <visual>
-        <origin rpy="0 1.5707 1.5707" xyz="0 0 0"/>
+        <origin rpy="1.570796 0 0" xyz="0 0 0"/>
         <geometry>
           <cylinder length="${wheel_width}" radius="${wheel_radius}"/>
@@ -18,14 +18,14 @@
       </visual>
       <collision>
-        <origin rpy="0 1.5707 1.5707" xyz="0 0 0"/>
+        <origin rpy="1.570796 0 0" xyz="0 0 0"/>
         <geometry>
           <cylinder length="${wheel_width}" radius="${wheel_radius}"/>
         </geometry>
       </collision>
-    <inertial>
-      <origin rpy="0 1.5707 1.5707" xyz="0 0 0"/>
-      <mass value="0.5" />
-      <inertia ixx="0.000172561667" ixy="0.0" ixz="0.0" iyy="0.000172561667" iyz="0.0" izz="0.00030976" />
-    </inertial>
+      <inertial>
+            <mass value="0.25"/>
+            <origin rpy="1.570796 0 0" xyz="0 0 0"/>
+            <inertia ixx="0.000058" ixy="0" ixz="0" iyy="0.000058" iyz="0" izz="0.000050"/>
+        </inertial>
   </link>
 </xacro:macro>

Commit message: Created the two robot spawn file

File: xacro/barista_robot_model.urdf.xacro (robot description, xacro)
@@ -1,4 +1,4 @@
 <?xml version="1.0"?>
-<robot name="morty" xmlns:xacro="http://ros.org/wiki/xacro">
+<robot name="barista_bot" xmlns:xacro="http://ros.org/wiki/xacro">
 <xacro:include filename="$(find barista_robot_description)/xacro/wheel.xacro" />
 <xacro:include filename="$(find barista_robot_description)/xacro/standoff.xacro" />
@@ -6,4 +6,7 @@
 <xacro:include filename="$(find barista_robot_description)/xacro/cup_holder_tray.xacro" />
 <xacro:include filename="$(find barista_robot_description)/xacro/laser_scanner.xacro" />
+<xacro:arg name="r_n" default="barista_bot"/>
+<xacro:property name="robot_name" value="$(arg r_n)"/>
+<xacro:property name="morty" value="morty"/>
 <xacro:property name="base_link_radius" value="0.178"/>
 <xacro:property name="base_link_length" value="0.155"/>
@@ -14,7 +17,10 @@
         <cylinder length="${base_link_length}" radius="${base_link_radius}" />
       </geometry>
-      <material name="red">
-        <color rgba="1.0 0.0 0.0 1"/>
-      </material>
+      <xacro:if value="${robot_name == morty}">
+      <material name="blue"/>
+      </xacro:if>
+      <xacro:unless value="${robot_name == morty}">
+      <material name="red"/>
+      </xacro:unless>
     </visual>
     <collision>
@@ -134,10 +140,24 @@
         <material>Gazebo/Black</material>
     </gazebo>
+    <xacro:if value="${robot_name == morty}">
 <gazebo reference="base_link">
-        <material>Gazebo/Red</material>
-    </gazebo>
+        <material>Gazebo/Blue</material>
+    </gazebo>
+    </xacro:if>
+  <xacro:unless value="${robot_name == morty}">
+  <gazebo reference="base_link">
+    <material>Gazebo/Red</material>
+  </gazebo>
+  </xacro:unless>
+<xacro:if value="${robot_name == morty}">
 <gazebo reference="cup_holder">
-        <material>Gazebo/Red</material>
-    </gazebo>
+        <material>Gazebo/Blue</material>
+    </gazebo>
+    </xacro:if>
+  <xacro:unless value="${robot_name == morty}">
+  <gazebo reference="cup_holder">
+    <material>Gazebo/Red</material>
+  </gazebo>
+  </xacro:unless>
 <gazebo reference="rod_a">
         <material>Gazebo/White</material>
@@ -158,7 +178,26 @@
         <preserveFixedJoint>true</preserveFixedJoint>
     </gazebo>
+<!-- Joint State Plugin -->
+  <gazebo>
+    <plugin name="joint_state" filename="libgazebo_ros_joint_state_publisher.so">
+      <ros>
+          <namespace>/${robot_name}</namespace>
+          <remapping>~/out:=joint_states</remapping>
+      </ros>
+      <update_rate>30</update_rate>
+      <joint_name>base_link_to_left_wheel</joint_name>
+      <joint_name>base_link_to_right_wheel</joint_name>
+      <joint_name>base_link_to_front_caster</joint_name>
+      <joint_name>base_link_to_back_caster</joint_name>
+      <joint_name>base_link_to_cup_holder</joint_name>
+    </plugin>
+  </gazebo>
  <!-- Differential drive -->
   <gazebo>
     <plugin filename="libgazebo_ros_diff_drive.so" name="differential_drive_controller">
+      <ros>
+        <namespace>/${robot_name}</namespace>
+        <remapping>~/out:=cmd_vel</remapping>
+      </ros>
       <!-- wheels -->
       <left_joint>base_link_to_left_wheel</left_joint>
@@ -173,6 +212,6 @@
       <publish_odom>true</publish_odom>
       <publish_odom_tf>true</publish_odom_tf>
-      <odometry_frame>odom</odometry_frame>
-      <robot_base_frame>base_link</robot_base_frame>
+      <odometry_frame>${robot_name}/odom</odometry_frame>
+      <robot_base_frame>${robot_name}/base_link</robot_base_frame>
     </plugin>
   </gazebo>

File: xacro/laser_scanner.xacro (robot description, xacro)
@@ -41,7 +41,9 @@
           <plugin name="laser" filename="libgazebo_ros_ray_sensor.so">
             <ros>
+              <namespace>/${robot_name}</namespace>
               <remapping>~/out:=scan</remapping>
             </ros>
             <output_type>sensor_msgs/LaserScan</output_type>
+             <frame_name>${robot_name}/hokuyo_sensor</frame_name>
           </plugin>
       </sensor>

Commit message: Did some changes to the two robot spawn. The rviz dosent show the two robots unless the file is selected in open config with the file name barista_two_bot

File: xacro/barista_robot_model.urdf.xacro (robot description, xacro)
@@ -11,4 +11,5 @@
 <xacro:property name="base_link_radius" value="0.178"/>
 <xacro:property name="base_link_length" value="0.155"/>
+<xacro:property name="include_laser" value="true"/>
 <!-- base_link -->
 <link name="base_link">
@@ -55,18 +56,18 @@
 <xacro:cup_holder cup_holder_name="cup_holder" />
 <!-- joints -->
-  <joint name="base_link_to_left_wheel" type="fixed">
+  <joint name="base_link_to_left_wheel" type="continuous">
     <origin rpy="0 0 0" xyz="0 0.145 -0.0775"/>
     <child link="left_wheel"/>
     <parent link="base_link"/>
-    <axis rpy="0 0 0" xyz="0 0 1"/>
+    <axis rpy="0 0 0" xyz="0 1 0"/>
     <limit effort="1000" velocity="100"/>
     <joint_properties damping="1.0" friction="1.0"/>
   </joint>
-  <joint name="base_link_to_right_wheel" type="fixed">
+  <joint name="base_link_to_right_wheel" type="continuous">
     <origin rpy="0 0 0" xyz="0 -0.145 -0.0775"/>
     <child link="right_wheel"/>
     <parent link="base_link"/>
-    <axis rpy="0 0 0" xyz="0 0 1"/>
-    <limit effort="1000" velocity="100"/>
+    <axis rpy="0 0 0" xyz="0 1 0"/>
+    <limit effort="1000" velocity="1000"/>
     <joint_properties damping="1.0" friction="1.0"/>
   </joint>
@@ -110,5 +111,10 @@
     <origin xyz="0 0 0.330" rpy="0 0 0"/>
   </joint>
-  <xacro:laser_scanner include_laser="True" />
+  <joint name="base_link_to_laser_sensor" type="fixed">
+    <origin xyz="0.130 0 0.0775" rpy="0 0 0"/>
+    <parent link="base_link"/>
+    <child link="laser_sensor"/>
+  </joint>
+   <xacro:laser_scanner robot_name="${robot_name}" include_laser="${include_laser}"/>
 <!-- gazebo references -->
   <gazebo reference="right_wheel">
@@ -176,4 +182,7 @@
     </gazebo>
 <gazebo reference="base_link_to_back_caster">
+        <preserveFixedJoint>true</preserveFixedJoint>
+    </gazebo>
+<gazebo reference="base_link_to_laser_sensor">
         <preserveFixedJoint>true</preserveFixedJoint>
     </gazebo>

File: xacro/laser_scanner.xacro (robot description, xacro)
@@ -1,53 +1,74 @@
 <?xml version="1.0"?>
-<robot xmlns:xacro="http://ros.org/wiki/xacro">
-  <xacro:macro name="laser_scanner" params="include_laser:=true">
-    <xacro:if value="${include_laser}">
-      <link name="hokuyo_sensor">
-          <visual>
-          <origin rpy="0 0 0" xyz="0 0 -0.0025" />
-              <geometry>
-                  <mesh filename="package://barista_robot_description/meshes/hokuyo_ust_10lx.dae" scale="1 1 1"/>
-              </geometry>
-          </visual>
-      </link>
-      <joint name="hokuyo_sensor_to_base_link" type="fixed">
-          <origin rpy="0 0 0" xyz="0.130 0 0.0775" />
-          <parent link="base_link" />
-          <child link="hokuyo_sensor" />
-      </joint>
-      <gazebo reference="hokuyo_sensor">
-          <material>Gazebo/Black</material>
-      </gazebo>
-    <gazebo reference="hokuyo_sensor">
-      <sensor name="ray" type="ray">
-          <pose>0 0 0 0 0 0</pose>
-          <ray>
-            <scan>
-              <horizontal>
-                <samples>720</samples>
-                <resolution>1.0</resolution>
-                <min_angle>-3.14</min_angle>
-                <max_angle>3.14</max_angle>
-              </horizontal>
-            </scan>
-            <range>
-              <min>0.1</min>
-              <max>5.0</max>
-            </range>
-          </ray>
-          <always_on>true</always_on>
-          <visualize>true</visualize>
-          <update_rate>100.0</update_rate>
-          <plugin name="laser" filename="libgazebo_ros_ray_sensor.so">
-            <ros>
-              <namespace>/${robot_name}</namespace>
-              <remapping>~/out:=scan</remapping>
-            </ros>
-            <output_type>sensor_msgs/LaserScan</output_type>
-             <frame_name>${robot_name}/hokuyo_sensor</frame_name>
-          </plugin>
-      </sensor>
-    </gazebo>
-    </xacro:if>
-  </xacro:macro>
+<robot xmlns:xacro="http://www.ros.org/wiki/xacro">
+    <xacro:macro name="laser_scanner" params="robot_name include_laser:=true">
+        <xacro:if value="${include_laser}">
+            <!-- Laser Sensor -->
+            <link name="laser_sensor">
+                <visual>
+                    <origin rpy="0 0 0" xyz="0 0 0"/>
+                    <geometry>
+                        <mesh filename="package://barista_robot_description/meshes/hokuyo.dae" scale="1 1 1"/>
+                    </geometry>
+                </visual>
+                <inertial>
+                    <mass value="0.160"/>
+                    <origin rpy="0 0 0" xyz="0 0 0"/>
+                    <inertia ixx="0.000099" ixy="0" ixz="0" iyy="0.000099" iyz="0" izz="0.000066"/>
+                </inertial>
+                <collision>
+                    <origin rpy="0 0 0" xyz="0 0 0"/>
+                    <geometry>
+                        <box size="0.050 0.050 0.070"/>
+                    </geometry>
+                </collision>
+            </link>
+            <!-- Laser Frame-->
+            <link name="laser_frame">
+                <inertial>
+                    <mass value="0.0001"/>
+                    <inertia ixx="0.0001" ixy="0.0" ixz="0.0" iyy="0.0001" iyz="0.0" izz="0.0001"/>
+                </inertial>
+            </link>
+            <!-- Laser Sensor - Laser Frame -->
+            <joint name="laser_sensor_to_laser_frame" type="fixed">
+                <parent link="laser_sensor"/>
+                <child link="laser_frame"/>
+                <origin xyz="0 0 0.060" rpy="0 0 0"/>
+            </joint>
+            <gazebo reference="laser_sensor_to_laser_frame">
+                <preserveFixedJoint>true</preserveFixedJoint>
+            </gazebo>
+            <!-- Laser Sensor Plugin -->
+            <gazebo reference="laser_frame">
+                <sensor name="${robot_name}_sensor_ray" type="ray">
+                    <pose>0 0 0 0 0 0</pose>
+                    <ray>
+                        <scan>
+                            <horizontal>
+                            <samples>200</samples>
+                            <resolution>1.0</resolution>
+                            <min_angle>-3.14</min_angle>
+                            <max_angle>3.14</max_angle>
+                            </horizontal>
+                        </scan>
+                        <range>
+                            <min>0.025</min>
+                            <max>5.0</max>
+                        </range>
+                    </ray>
+                    <always_on>true</always_on>
+                    <visualize>false</visualize>
+                    <update_rate>10.0</update_rate>
+                    <plugin name="${robot_name}_laser" filename="libgazebo_ros_ray_sensor.so">
+                        <ros>
+                            <namespace>/${robot_name}</namespace>
+                            <remapping>~/out:=scan</remapping>
+                        </ros>
+                        <frame_name>${robot_name}/laser_frame</frame_name>
+                        <output_type>sensor_msgs/LaserScan</output_type>
+                    </plugin>
+                </sensor>
+            </gazebo>
+        </xacro:if>
+    </xacro:macro>
 </robot>
